File: schematic/motor_controller/motor_controller.kicad_sch (KiCad schematic)
At the start: 13 parts, among them J1 Micro_SD_Card, J2 Conn_01x19_Pin, J3 Conn_01x19_Pin, U1 AMS1117-5.0, U2 74LVC125APW_118

Commit message: Final schematic for review
Parts:
- removed J2, J3: Conn_01x19_Pin, Connector_Molex:Molex_SL_171971-0019_1x19_P2.54mm_Vertical, symbol Connector:Conn_01x19_Pin
- added C5, C6: 10u, Capacitor_SMD:C_1210_3225Metric, symbol Device:C
- added C7: 100u, Capacitor_SMD:C_Elec_6.3x5.8, symbol Device:C
- added C8: 0.05u, Capacitor_SMD:C_1206_3216Metric, symbol Device:C
- added C9: 150u, Capacitor_SMD:C_Elec_6.3x7.7, symbol Device:C
- added J2, J4: Conn_01x20_Pin, Connector_PinHeader_1.00mm:PinHeader_1x20_P1.00mm_Vertical, symbol Connector:Conn_01x20_Pin
- added J3: Conn_01x01_Pin, Connector_PinHeader_1.00mm:PinHeader_1x01_P1.00mm_Vertical, symbol Connector:Conn_01x01_Pin
- added R5: 10, Resistor_SMD:R_0402_1005Metric, symbol Device:R
- added RV1: 10k, Potentiometer_THT:Potentiometer_Alpha_RD901F-40-00D_Single_Vertical, symbol Device:R_Potentiometer
- added U3: LM386, Package_DIP:DIP-8_W7.62mm, symbol Amplifier_Audio:LM386
- C1, C2, C3, C4: footprint (none) -> Capacitor_SMD:C_0402_1005Metric
- R1, R2, R3, R4: footprint (none) -> Resistor_SMD:R_0402_1005Metric
- U1: footprint Connector_Card:microSD_HC_Molex_104031-0811 -> Symbol:SOT229P700X180-4N
- U2: footprint TSSOP14_SOT402-1_NEX -> Symbol:IC_74LVC125APW_118
Connections:
- net +5V: now also U2.11 (4Y), J4.19 (Pin_19), J4.5 (Pin_5), U3.6 (V+)
- net GND: now also J1.6 (VSS), R2.1, U2.12 (4A), J2.20 (Pin_20), J4.20 (Pin_20), R5.2, RV1.3, U3.2 (-), U3.4 (GND)
- net CS: now reaches R1.1
- net CS: now also J4.8 (Pin_8)
- net MOSI: now reaches R3.1
- net MOSI: now also J4.6 (Pin_6)
- net SCK: now reaches R4.1
- net SCK: now also J4.7 (Pin_7)
- new net: C8.1, R5.1
- new net: C7.1, C8.2, C9.1, U3.5
- new net: C6.1, U3.1 (GAIN)
- new net: C6.2, U3.8 (GAIN)
- new net: C5.2, RV1.1
- new net: RV1.2, U3.3 (+)
- new net Audio: C5.1, J2.1 (Pin_1)
- new net speaker: C7.2, C9.2, J3.1 (Pin_1)
Other:
- note added: "Digital pins"

Commit message: Final schematic reviewed
Parts:
- J2, J4: footprint Connector_PinHeader_1.00mm:PinHeader_1x20_P1.00mm_Vertical -> Connector_PinHeader_2.54mm:PinHeader_1x20_P2.54mm_Vertical
Changed lines of the file:
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@@
 			)
 		)
-		(property "Footprint" "Connector_PinHeader_1.00mm:PinHeader_1x20_P1.00mm_Vertical"
+		(property "Footprint" "Connector_PinHeader_2.54mm:PinHeader_1x20_P2.54mm_Vertical"
 			(at 95.25 57.15 0)
 			(effects
@@
 			)
 		)
-		(property "Footprint" "Connector_PinHeader_1.00mm:PinHeader_1x20_P1.00mm_Vertical"
+		(property "Footprint" "Connector_PinHeader_2.54mm:PinHeader_1x20_P2.54mm_Vertical"
 			(at 137.16 57.15 0)
 			(effects
